File: cad/TPadTabletBattery.sch (EAGLE design)
At the start: 105 parts, among them J1 MOLEX-MINI-FIT-JR-2POS-RA, J2 USB IN, J3 POWER_JACKPTH, J4 USBA-THRU-UE27-AC54-100, Q1 NCH, Q2 PCH, U1 MCP73833-AMI/UN, U2 STM-LOW-SWITCH-VNL5050N3TR-E, U3 TPS43000_PW_16, U4 PIC24FJ256GB206, U5 MICROCHIP-MINI-DRIVER-MCP1416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, U6 TI-AUDIOAMP-LM48100Q, U7 TI-AUDIOAMP-LM48100Q, U8 TI-AUDIOAMP-LM48100Q, U9 TI-AUDIOAMP-LM48100Q

Commit message: USB OTG board version updated
Parts:
- removed J4: USBA-THRU-UE27-AC54-100, Craig:USBA-THRU-UE27-AC54-100
- added C40, C41, C42, C43: 10uF, MCP73833_QFN_v1.0:MICROBUILDER_CAP_CERAMIC0805
- added C44, C45, C46, C47: 0.1uF, MCP73833_QFN_v1.0:MICROBUILDER_CAP_CERAMIC0603
- added C48: 47uF, SparkFun-Capacitors:CAP1210
- added JP1, JP10, JP14: (no value), SparkFun-Connectors:M06SIP
- added LED6: F1, MCP73833_QFN_v1.0:MICROBUILDER_LED0603
- added LED7: F2, MCP73833_QFN_v1.0:MICROBUILDER_LED0603
- added LED8: F3, MCP73833_QFN_v1.0:MICROBUILDER_LED0603
- added LED9: F4, MCP73833_QFN_v1.0:MICROBUILDER_LED0603
- added U$1: USBA-THRU-PLUG, Craig:USBA-THRU-PLUG
- C28, C29, C31, C32, C34, C35, C37, C38: value 0.1uF -> 0.47uF
- C4, C5: value 330UF_POSCAP -> 330uF
- L1: value .82UH_INDUCTOR-IHLP3232DZERR82M01 -> .82uH
- LED5: value GREEN -> +5V
Connections:
- removed net N$9: R18.2, R28.1
- removed net SCL2: R21.2, U4.SCL2/RP17/GD5/CN18/RF5, U8.SCL, U9.SCL
- removed net SDA2: R22.2, U4.SDA2/RP10/GD4/CN17/RF4, U8.SDA, U9.SDA
- removed net USBID: U4.RP16/USBID/CN71/RF3
- new net 5V_USB: LED5.A, U$1.5V, U$6.5V, U4.VBUS/RF7
- new net N$6: R28.2, U4.!MCLR
- new net SCL0: R19.2, U4.SCL1/RP3/GD6/CN55/RD10, U6.SCL, U7.SCL
- new net SDA0: R20.2, U4.DPLN/SDA1/RP4/GD8/CN54/RD9, U6.SDA, U7.SDA
- net +3V3: now also C48.1
- net D+: now also U$1.D+; no longer J4.D+
- net D-: now also U$1.D-; no longer J4.D-
- net FAULT1: now also LED6.A
- net FAULT2: now also LED7.A
- net FAULT3: now also LED8.A
- net FAULT4: now also LED9.A
- net GND: now also C40.P$2, C41.P$2, C42.P$2, C43.P$2, C44.P$2, C45.P$2, C46.P$2, C47.P$2, C48.2, LED6.C, LED7.C, LED8.C, LED9.C, U$1.GND, U$1.S1, U$1.S2, U4.RP16/USBID/CN71/RF3; no longer J4.GND, J4.S1, J4.S2
- net MCLR: now also R18.2, R28.1; no longer R28.2, U4.!MCLR
- net PIN24: now also JP1.6
- net PIN25: now also JP1.5
- net PIN26: now also JP1.4
- net PIN27: now also JP1.3
- net PIN28: now also JP1.2
- net PIN29: now also JP1.1
- net PIN37: now also JP10.6
- net PIN38: now also JP10.5
- net PIN39: now also JP10.4
- net PIN40: now also JP10.3
- net PIN41: now also JP10.2
- net PIN42: now also JP10.1
- net PIN43: now also JP14.6
- net PIN44: now also JP14.5
- net PIN45: now also JP14.4
- net PIN46: now also JP14.3
- net SCL1: now also JP14.1, R21.2, U4.SCL2/RP17/GD5/CN18/RF5, U8.SCL, U9.SCL; no longer R19.2, U4.SCL1/RP3/GD6/CN55/RD10, U6.SCL, U7.SCL
- net SDA1: now also JP14.2, R22.2, U4.SDA2/RP10/GD4/CN17/RF4, U8.SDA, U9.SDA; no longer R20.2, U4.DPLN/SDA1/RP4/GD8/CN54/RD9, U6.SDA, U7.SDA
- net VCC: now also C40.P$1, C41.P$1, C42.P$1, C43.P$1, C44.P$1, C45.P$1, C46.P$1, C47.P$1; no longer J4.5V, LED5.A, U$6.5V, U4.VBUS/RF7
Other:
- note removed: "Aux Battery Connection"
- note removed: "Ytai Ben-tsvi"
- note removed: "revised by A.Weiss"
